File: Projects/Ebike/schwinn-ecotour/schwinn-ecotour.kicad_sch (KiCad schematic)
At the start: 18 parts, among them J1 5vin, J2 wheel sensor, J3 24vin, J4 leftsw, J5 rightsw, J6 brakesw, J7 lightsw, J8 AnalogIn, J9 serial, SW1 Up / +, SW2 Down / -, SW3 Enter, SW4 Back, SW5 Home

Commit message: update pcb layout (forgot to hit save)
Parts:
- SW5: value Home -> toggle
Changed lines of the file:
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@@
       (effects (font (size 1.27 1.27)))
     )
-    (property "Value" "Home" (at 133.35 80.01 0)
+    (property "Value" "toggle" (at 133.35 80.01 0)
       (effects (font (size 1.27 1.27)))
     )
