File: Projects/Ebike/schwinn-ecotour/schwinn-ecotour.kicad_sch (KiCad schematic)
At the start: 21 parts, among them J1 5vin, J11 misclights, J12 Conn_01x02_Pin, J2 Conn_01x03_Pin, J3 24vin, J4 Conn_01x11_Socket, J5 headlight, J6 brakesw, J8 AnalogIn, J9 serial, SW1 Up / +, SW2 Down / -, SW3 Enter, SW4 turn signals, SW5 headlights, U1 SM351LT, U7 8255

Commit message: more schematic & pcb work
Parts:
- removed J4: Conn_01x11_Socket, Connector_PinSocket_1.27mm:PinSocket_1x11_P1.27mm_Vertical, symbol Connector:Conn_01x11_Socket
- removed J8: AnalogIn, Connector_PinHeader_2.54mm:PinHeader_1x02_P2.54mm_Vertical, symbol Connector:Conn_01x02_Socket
- removed U7: 8255, Package_DIP:DIP-40_W15.24mm, symbol Interface:8255
Connections:
- net at A1.19 (A0): now also SW5.1
- net at A1.20 (A1): now also SW5.2
- net at J11.2 (Pin_2), J6.2 (Pin_2): now also A1.22 (A3)
- net at SW5.4: now also A1.21 (A2)
- net at SW3.1: now also A1.13 (D10)
- net at DS1.11 (D4): now also A1.7 (D4)
- net at DS1.12 (D5): now also A1.8 (D5)
- net at DS1.13 (D6): now also A1.9 (D6)
- net at DS1.14 (D7): now also A1.10 (D7)
- net at DS1.4 (RS): now also A1.6 (D3)
- net at DS1.6 (E): now also A1.5 (D2)
- net at A1.11 (D8): now also SW1.1
- net at A1.12 (D9): now also SW2.1
- net at A1.14 (D11): now also SW4.4 (A)
- net at A1.15 (D12): now also SW4.6 (C)
