File: Projects/Ebike/schwinn-ecotour/schwinn-ecotour.kicad_pcb (KiCad board)
At the start: 2 copper layers, 17 parts, among them J1 5vin, J2 wheel sensor, J4 leftsw, J5 rightsw, J6 brakesw, J7 lightsw, J8 AnalogIn, J9 serial, SW1 Up / +, SW2 Down / -, SW3 Enter, SW4 Back, SW5 Home

Commit message: update pcb layout (forgot to hit save)
Parts:
- moved A1 26.9 mm to (116.8, 61.0), turned to -90 degrees
- moved J4 5.08 mm to (170.2, 43.2)
- moved J5 5.08 mm to (165.1, 43.2)
Routing:
- net GND: track 0.00 -> 208.8 mm
- net Net-(A1-D9): track 0.00 -> 194.7 mm
- net Net-(A1-D3): track 0.00 -> 191.5 mm
- net Net-(A1-D6): track 0.00 -> 180.1 mm
- net Net-(A1-D5): track 0.00 -> 98.0 mm
- net -5V: track 0.00 -> 82.2 mm
- net Net-(DS1-VO): track 0.00 -> 72.1 mm
- net Net-(A1-D4): track 0.00 -> 70.3 mm
- net Net-(A1-A1): track 0.00 -> 61.3 mm
- net Net-(A1-A0): track 0.00 -> 60.8 mm
- net Net-(A1-D10): track 0.00 -> 32.6 mm
- net Net-(A1-D8): track 0.00 -> 25.2 mm
- net Net-(A1-D2): track 0.00 -> 14.2 mm
- net (no net): track 0.00 -> 2.58 mm
- net unconnected-(A1-~{RESET}-Pad28): track 0.00 -> 2.08 mm

Commit message: more schematic & pcb work
Parts:
- removed J2: wheel sensor, Connector_PinHeader_2.54mm:PinHeader_1x02_P2.54mm_Vertical
- removed J4: leftsw, Connector_PinHeader_2.54mm:PinHeader_1x02_P2.54mm_Vertical
- removed J7: lightsw, Connector_PinHeader_2.54mm:PinHeader_1x02_P2.54mm_Vertical
- removed J8: AnalogIn, Connector_PinHeader_2.54mm:PinHeader_1x02_P2.54mm_Vertical
- added J11: misclights, Connector_PinHeader_1.27mm:PinHeader_1x03_P1.27mm_Horizontal, F.Cu at (152.4, 71.1)
- added U1: SM351LT, Connector_PinHeader_1.27mm:PinHeader_1x03_P1.27mm_Horizontal, F.Cu at (129.5, 71.1)
- J5: value rightsw -> headlight; footprint Connector_PinHeader_2.54mm:PinHeader_1x02_P2.54mm_Vertical -> Connector_PinHeader_1.27mm:PinHeader_1x03_P1.27mm_Horizontal
- J6, RV1: moved to B.Cu
- RV2: footprint Potentiometer_THT:Potentiometer_ACP_CA14-H2,5_Horizontal -> Potentiometer_THT:Potentiometer_Alpha_RD901F-40-00D_Single_Vertical_CircularHoles
- SW4: value Back -> turn signals; footprint Button_Switch_THT:SW_PUSH_6mm_H4.3mm -> Connector_PinSocket_1.27mm:PinSocket_2x03_P1.27mm_Horizontal
- SW5: value Home -> headlights; footprint Connector_PinHeader_2.54mm:PinHeader_1x02_P2.54mm_Vertical -> Connector_PinHeader_1.27mm:PinHeader_2x04_P1.27mm_Vertical
- moved RV2 114.1 mm to (215.4, 68.6)
- moved A1 92.4 mm to (195.6, 109.2), turned to 0 degrees
- moved J9 81.8 mm to (193.0, 109.2), turned to 180 degrees
- moved SW1 46.2 mm to (217.0, 99.3)
- moved J6 41.7 mm to (144.8, 68.6), turned to 180 degrees
- moved SW5 30.6 mm to (180.3, 66.0)
- moved J5 27.9 mm to (165.1, 71.1), turned to 90 degrees
- moved SW4 25.9 mm to (189.2, 69.8), turned to -90 degrees
- moved DS1 25.4 mm to (117.9, 78.6)
- moved J1 22.9 mm to (111.8, 66.0)
- moved SW3 22.5 mm to (217.0, 81.3)
- moved SW2 21.3 mm to (217.0, 89.5)
- moved RV1 19.2 mm to (121.9, 69.3)
Connections:
- A1 pad 10: unconnected-(A1-D7-Pad10) -> Net-(A1-D7)
- A1 pad 14: unconnected-(A1-D11-Pad14) -> Net-(A1-D11)
- A1 pad 15: unconnected-(A1-D12-Pad15) -> Net-(A1-D12)
- A1 pad 16: unconnected-(A1-D13-Pad16) -> Net-(A1-D13)
- A1 pad 21: unconnected-(A1-A2-Pad21) -> Net-(A1-A2)
- A1 pad 22: unconnected-(A1-A3-Pad22) -> Net-(A1-A3)
- DS1 pad 10: Net-(A1-D6) -> unconnected-(DS1-D3-Pad10)
- DS1 pad 11: unconnected-(DS1-D4-Pad11) -> Net-(A1-D4)
- DS1 pad 12: unconnected-(DS1-D5-Pad12) -> Net-(A1-D5)
- DS1 pad 13: unconnected-(DS1-D6-Pad13) -> Net-(A1-D6)
- DS1 pad 14: unconnected-(DS1-D7-Pad14) -> Net-(A1-D7)
- DS1 pad 4: Net-(A1-D2) -> Net-(A1-D3)
- DS1 pad 6: Net-(A1-D8) -> Net-(A1-D2)
- DS1 pad 7: Net-(A1-D3) -> unconnected-(DS1-D0-Pad7)
- DS1 pad 8: Net-(A1-D4) -> unconnected-(DS1-D1-Pad8)
- DS1 pad 9: Net-(A1-D5) -> unconnected-(DS1-D2-Pad9)
- J5 pad 1: Net-(A1-D10) -> Net-(J5-Pin_1)
- J5 pad 2: Net-(A1-D4) -> Net-(J5-Pin_2)
- J6 pad 1: Net-(A1-D10) -> GND
- J6 pad 2: Net-(A1-D5) -> Net-(A1-A3)
- SW1 pad 1: Net-(A1-D9) -> Net-(A1-D8)
- SW1 pad 2: Net-(A1-D3) -> GND
- SW2 pad 2: Net-(A1-D4) -> GND
- SW3 pad 1: Net-(A1-D9) -> Net-(A1-D10)
- SW3 pad 2: Net-(A1-D5) -> GND
- SW4 pad 1: Net-(A1-D9) -> Net-(J11-Pin_1)
- SW4 pad 2: Net-(A1-D6) -> -5V
- SW5 pad 1: Net-(A1-D9) -> Net-(A1-A0)
- SW5 pad 2: Net-(A1-D2) -> Net-(A1-A1)
Routing:
- net -5V: track 82.2 -> 421.1 mm
- net Net-(A1-D13): track 0.00 -> 281.3 mm
- net Net-(A1-D9): track 194.7 -> 31.5 mm
- net Net-(DS1-LED(+)): track 0.00 -> 130.7 mm, vias 0 -> 1
- net Net-(A1-D3): track 191.5 -> 77.2 mm
- net Net-(A1-D6): track 180.1 -> 67.1 mm
- net Net-(A1-A3): track 0.00 -> 73.8 mm
- net Net-(A1-D2): track 14.2 -> 86.5 mm
- net Net-(A1-D7): track 0.00 -> 69.3 mm
- net Net-(DS1-VO): track 72.1 -> 5.28 mm
- net Net-(J11-Pin_1): track 0.00 -> 47.0 mm, vias 0 -> 1
- net Net-(J11-Pin_3): track 0.00 -> 43.0 mm, vias 0 -> 1
- net Net-(A1-A2): track 0.00 -> 37.1 mm
- net Net-(A1-D5): track 98.0 -> 66.5 mm
- net GND: track 208.8 -> 178.3 mm
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- added copper zone on F.Cu, net GND
